Commit message: update from manefest to package.xml

File: urdf/computers/m200_jt2.urdf.xacro (robot description, xacro)
@@ -1,5 +1,5 @@
 <?xml version="1.0"?>
 <robot name="computers" xmlns:xacro="http://ros.org/wiki/xacro">
-	<!--<xacro:include filename="$(find tegraBot_description)/urdf/common_properties.urdf.xacro"/>-->
+	<!--<xacro:include filename="$(find tegrabot_description)/urdf/common_properties.urdf.xacro"/>-->
   <xacro:macro name="computers" params="parent">
   <!--
@@ -18,5 +18,5 @@
         <origin xyz="0 0 0.0" rpy="0 0 0"/>
         <geometry>
-          <mesh filename="package://tegraBot_description/meshes/computers/m200_jt2.dae" />
+          <mesh filename="package://tegrabot_description/meshes/computers/m200_jt2.dae" />
         </geometry>
 		<material name="material_blue"/>

File: urdf/kobuki.urdf.xacro (robot description, xacro)
@@ -7,6 +7,6 @@
  -->
 <robot name="kobuki" xmlns:xacro="http://ros.org/wiki/xacro">
-  <xacro:include filename="$(find tegraBot_description)/urdf/common_properties.urdf.xacro"/>
-  <!--<xacro:include filename="$(find tegraBot_description)/urdf/kobuki_gazebo.urdf.xacro"/>-->
+  <xacro:include filename="$(find tegrabot_description)/urdf/common_properties.urdf.xacro"/>
+  <!--<xacro:include filename="$(find tegrabot_description)/urdf/kobuki_gazebo.urdf.xacro"/>-->
   <!-- Kobuki -->
   <xacro:macro name="kobuki">
@@ -30,5 +30,5 @@
         <geometry>
           <!-- new mesh -->
-          <mesh filename="package://tegraBot_description/meshes/main_body.dae" />
+          <mesh filename="package://tegrabot_description/meshes/main_body.dae" />
         </geometry>
         <origin xyz="0.001 0 0.05199" rpy="0 0 0"/>
@@ -65,5 +65,5 @@
       <visual>
         <geometry>
-          <mesh filename="package://tegraBot_description/meshes/wheel.dae"/>
+          <mesh filename="package://tegrabot_description/meshes/wheel.dae"/>
         </geometry>
         <origin xyz="0 0 0" rpy="0 0 0"/>
@@ -92,5 +92,5 @@
       <visual>
         <geometry>
-          <mesh filename="package://tegraBot_description/meshes/wheel.dae"/>
+          <mesh filename="package://tegrabot_description/meshes/wheel.dae"/>
         </geometry>
         <origin xyz="0 0 0" rpy="0 0 0"/>

File: urdf/sensors/astra.urdf.xacro (robot description, xacro)
@@ -1,6 +1,6 @@
 <?xml version="1.0"?>
 <robot name="sensor_astra" xmlns:xacro="http://ros.org/wiki/xacro">
-	<!--<xacro:include filename="$(find tegraBot_description)/urdf/turtlebot_gazebo.urdf.xacro"/>-->
-  <xacro:include filename="$(find tegraBot_description)/urdf/tegraBot_properties.urdf.xacro"/>
+	<!--<xacro:include filename="$(find tegrabot_description)/urdf/turtlebot_gazebo.urdf.xacro"/>-->
+  <xacro:include filename="$(find tegrabot_description)/urdf/tegraBot_properties.urdf.xacro"/>
   <!-- Xacro properties -->
   <xacro:property name="astra_cam_py" value="-0.008"/>
@@ -33,5 +33,5 @@
         <origin xyz="-0.04 0.02 -0.01" rpy="${M_PI/2} 0 ${M_PI/2}"/>
         <geometry>
-          <mesh filename="package://tegraBot_description/meshes/sensors/astra.dae" scale="${astra_dae_display_scale} ${astra_dae_display_scale} ${astra_dae_display_scale}"/>
+          <mesh filename="package://tegrabot_description/meshes/sensors/astra.dae" scale="${astra_dae_display_scale} ${astra_dae_display_scale} ${astra_dae_display_scale}"/>
         </geometry>
       </visual>

File: urdf/sensors/asus_xtion_pro.urdf.xacro (robot description, xacro)
@@ -33,5 +33,5 @@
         <origin xyz="-0.015 0.0035 0.004" rpy="0 0 0"/>
         <geometry>
-          <mesh filename="package://tegraBot_description/meshes/sensors/xtion_pro_camera.dae"/>
+          <mesh filename="package://tegrabot_description/meshes/sensors/xtion_pro_camera.dae"/>
         </geometry>
       </visual>
@@ -74,5 +74,5 @@
         <origin xyz="0 0 0" rpy="${-M_PI/2} 0 0"/>
         <geometry>
-          <mesh filename="package://tegraBot_description/meshes/sensors/xtion_pro_stack.dae"/>
+          <mesh filename="package://tegrabot_description/meshes/sensors/xtion_pro_stack.dae"/>
         </geometry>
       </visual>

File: urdf/sensors/asus_xtion_pro_offset.urdf.xacro (robot description, xacro)
@@ -33,5 +33,5 @@
         <origin xyz="-0.01 0 0" rpy="${-M_PI/2} -${M_PI} ${-M_PI/2}"/>
         <geometry>
-          <mesh filename="package://tegraBot_description/meshes/sensors/asus_xtion_pro_live.dae" scale="${M_SCALE} ${M_SCALE} ${M_SCALE}"/>
+          <mesh filename="package://tegrabot_description/meshes/sensors/asus_xtion_pro_live.dae" scale="${M_SCALE} ${M_SCALE} ${M_SCALE}"/>
         </geometry>
       </visual>

File: urdf/sensors/kinect.urdf.xacro (robot description, xacro)
@@ -27,5 +27,5 @@
        <origin xyz="0 0 0" rpy="0 0 ${M_PI/2}"/>
         <geometry>
-         <mesh filename="package://tegraBot_description/meshes/sensors/kinect.dae"/>
+         <mesh filename="package://tegrabot_description/meshes/sensors/kinect.dae"/>
         </geometry>
       </visual>

File: urdf/sensors/r200.urdf.xacro (robot description, xacro)
@@ -35,5 +35,5 @@
        <origin xyz="${-r200_bracket_end_width/2} ${r200_bracket_end_offset_py} ${r200_bracket_end_offset_pz}" rpy="0 0 ${-M_PI/2}"/>
         <geometry>
-         <mesh filename="package://tegraBot_description/meshes/sensors/r200_bracket_end.stl" scale="0.001 0.001 0.001"/>
+         <mesh filename="package://tegrabot_description/meshes/sensors/r200_bracket_end.stl" scale="0.001 0.001 0.001"/>
         </geometry>
         <xacro:insert_block name="material_dark_grey" />
@@ -50,5 +50,5 @@
        <origin xyz="0 0 0" rpy="0 0 ${M_PI/2}"/>
         <geometry>
-         <mesh filename="package://tegraBot_description/meshes/sensors/r200_bracket.stl" scale="0.001 0.001 0.001"/>
+         <mesh filename="package://tegrabot_description/meshes/sensors/r200_bracket.stl" scale="0.001 0.001 0.001"/>
         </geometry>
         <xacro:insert_block name="material_dark_grey" />
@@ -65,5 +65,5 @@
        <origin xyz="${r200_bracket_end_width/2} 0 ${-r200_bracket_end_offset_pz}" rpy="0 0 ${M_PI/2}"/>
         <geometry>
-         <mesh filename="package://tegraBot_description/meshes/sensors/r200_bracket_end.stl" scale="0.001 0.001 0.001"/>
+         <mesh filename="package://tegrabot_description/meshes/sensors/r200_bracket_end.stl" scale="0.001 0.001 0.001"/>
         </geometry>
         <xacro:insert_block name="material_dark_grey" />
@@ -80,5 +80,5 @@
        <origin xyz="0 0 0" rpy="${M_PI/2} 0 ${M_PI/2}"/>
         <geometry>
-         <mesh filename="package://tegraBot_description/meshes/sensors/r200.dae" />
+         <mesh filename="package://tegrabot_description/meshes/sensors/r200.dae" />
         </geometry>
       </visual>

File: urdf/sensors/ydlidar_x4.urdf.xacro (robot description, xacro)
@@ -1,6 +1,6 @@
 <?xml version="1.0"?>
 <robot name="sensor_ydlidar" xmlns:xacro="http://ros.org/wiki/xacro">
-	<!--<xacro:include filename="$(find tegraBot_description)/urdf/turtlebot_gazebo.urdf.xacro"/>-->
-  <xacro:include filename="$(find tegraBot_description)/urdf/tegraBot_properties.urdf.xacro"/>
+	<!--<xacro:include filename="$(find tegrabot_description)/urdf/turtlebot_gazebo.urdf.xacro"/>-->
+  <xacro:include filename="$(find tegrabot_description)/urdf/tegraBot_properties.urdf.xacro"/>
   <!-- Parameterised in part by the values in tegraBot_properties.urdf.xacro -->
   <xacro:macro name="sensor_ydlidar" params="parent">
@@ -15,5 +15,5 @@
         <origin xyz="0 0 0" rpy="0 0 0"/>
         <geometry>
-          <mesh filename="package://tegraBot_description/meshes/sensors/ydlidar_x4.dae"/>
+          <mesh filename="package://tegrabot_description/meshes/sensors/ydlidar_x4.dae"/>
         </geometry>
       </visual>

File: urdf/stacks/hexagons.urdf.xacro (robot description, xacro)
@@ -4,5 +4,5 @@
  -->
 <robot name="stack_hexagons" xmlns:xacro="http://ros.org/wiki/xacro">
-  <xacro:include filename="$(find tegraBot_description)/urdf/common_properties.urdf.xacro"/>
+  <xacro:include filename="$(find tegrabot_description)/urdf/common_properties.urdf.xacro"/>
   <!-- Xacro properties -->
   <xacro:property name="M_SCALE" value="0.001"/>
@@ -19,5 +19,5 @@
         <origin xyz="0 0 0" rpy="0 0 0"/>
         <geometry>
-          <mesh filename="package://tegraBot_description/meshes/stacks/hexagons/pole_bottom.dae"/>
+          <mesh filename="package://tegrabot_description/meshes/stacks/hexagons/pole_bottom.dae"/>
         </geometry>
       </visual>
@@ -47,5 +47,5 @@
         <origin xyz="0 0 0" rpy="0 ${M_PI} 0"/>
         <geometry>
-          <mesh filename="package://tegraBot_description/meshes/stacks/hexagons/pole_middle.dae"/>
+          <mesh filename="package://tegrabot_description/meshes/stacks/hexagons/pole_middle.dae"/>
         </geometry>
       </visual>
@@ -75,5 +75,5 @@
         <origin xyz=" 0 0 0" rpy="0 0 0"/>
         <geometry>
-          <mesh filename="package://tegraBot_description/meshes/stacks/hexagons/pole_top.dae"/>
+          <mesh filename="package://tegrabot_description/meshes/stacks/hexagons/pole_top.dae"/>
         </geometry>
       </visual>
@@ -103,5 +103,5 @@
         <origin xyz="0 0 -0.01" rpy="0 0 0"/>
         <geometry>
-          <mesh filename="package://tegraBot_description/meshes/sensors/sensor_pole.dae" />
+          <mesh filename="package://tegrabot_description/meshes/sensors/sensor_pole.dae" />
         </geometry>
       </visual>
@@ -142,5 +142,5 @@
         <origin xyz="0 0 0" rpy="0 0 0"/>
         <geometry>
-          <mesh filename="package://tegraBot_description/meshes/stacks/hexagons/plate_bottom.dae"/>
+          <mesh filename="package://tegrabot_description/meshes/stacks/hexagons/plate_bottom.dae"/>
         </geometry>
       </visual>
@@ -172,5 +172,5 @@
         <origin xyz="0 0 0" rpy="0 0 0"/>
         <geometry>
-          <mesh filename="package://tegraBot_description/meshes/stacks/hexagons/plate_middle.dae"/>
+          <mesh filename="package://tegrabot_description/meshes/stacks/hexagons/plate_middle.dae"/>
         </geometry>
       </visual>
@@ -204,5 +204,5 @@
         <origin xyz="0 0 0" rpy="0 0 0"/>
         <geometry>
-          <mesh filename="package://tegraBot_description/meshes/stacks/hexagons/plate_top.dae"/>
+          <mesh filename="package://tegrabot_description/meshes/stacks/hexagons/plate_top.dae"/>
         </geometry>
       </visual>

File: urdf/stacks/tegraBot_stack.urdf.xacro (robot description, xacro)
@@ -4,5 +4,5 @@
  -->
 <robot name="stack_hexagons" xmlns:xacro="http://ros.org/wiki/xacro">
-  <xacro:include filename="$(find tegraBot_description)/urdf/common_properties.urdf.xacro"/>
+  <xacro:include filename="$(find tegrabot_description)/urdf/common_properties.urdf.xacro"/>
   <!-- Xacro properties -->
   <xacro:property name="M_SCALE" value="0.001"/>
@@ -19,5 +19,5 @@
         <origin xyz="0 0 0" rpy="0 0 0"/>
         <geometry>
-          <mesh filename="package://tegraBot_description/meshes/stacks/hexagons/pole_bottom.dae"/>
+          <mesh filename="package://tegrabot_description/meshes/stacks/hexagons/pole_bottom.dae"/>
         </geometry>
       </visual>
@@ -47,5 +47,5 @@
         <origin xyz="0 0 0" rpy="0 ${M_PI} 0"/>
         <geometry>
-          <mesh filename="package://tegraBot_description/meshes/stacks/hexagons/pole_middle.dae"/>
+          <mesh filename="package://tegrabot_description/meshes/stacks/hexagons/pole_middle.dae"/>
         </geometry>
       </visual>
@@ -76,5 +76,5 @@
         <origin xyz=" 0 0 0" rpy="0 0 0"/>
         <geometry>
-          <mesh filename="package://tegraBot_description/meshes/stacks/hexagons/pole_top.dae"/>
+          <mesh filename="package://tegrabot_description/meshes/stacks/hexagons/pole_top.dae"/>
         </geometry>
       </visual>
@@ -104,5 +104,5 @@
         <origin xyz="0 0 -0.01" rpy="0 0 0"/>
         <geometry>
-          <mesh filename="package://tegraBot_description/meshes/sensors/sensor_pole.dae" />
+          <mesh filename="package://tegrabot_description/meshes/sensors/sensor_pole.dae" />
         </geometry>
       </visual>
@@ -145,5 +145,5 @@
         <origin xyz="0 0 0" rpy="0 0 0"/>
         <geometry>
-          <mesh filename="package://tegraBot_description/meshes/stacks/hexagons/plate_bottom.dae"/>
+          <mesh filename="package://tegrabot_description/meshes/stacks/hexagons/plate_bottom.dae"/>
         </geometry>
       </visual>
@@ -175,5 +175,5 @@
         <origin xyz="0 0 0" rpy="0 0 0"/>
         <geometry>
-          <mesh filename="package://tegraBot_description/meshes/stacks/hexagons/plate_middle.dae"/>
+          <mesh filename="package://tegrabot_description/meshes/stacks/hexagons/plate_middle.dae"/>
         </geometry>
       </visual>
@@ -201,5 +201,5 @@
         <origin xyz="0 0 -0.01" rpy="0 0 0"/>
         <geometry>
-          <mesh filename="package://tegraBot_description/meshes/stacks/sensor_pole.dae" />
+          <mesh filename="package://tegrabot_description/meshes/stacks/sensor_pole.dae" />
         </geometry>
 		<material name="material_black"/>
@@ -234,5 +234,5 @@
         <origin xyz="0 0 0" rpy="0 0 0"/>
         <geometry>
-          <mesh filename="package://tegraBot_description/meshes/stacks/hexagons/plate_top.dae"/>
+          <mesh filename="package://tegrabot_description/meshes/stacks/hexagons/plate_top.dae"/>
         </geometry>
       </visual>

File: urdf/tegraBot.urdf.xacro (robot description, xacro)
@@ -11,11 +11,11 @@
 -->
 	<!--Following lines was copied from kobuki_hexagons_astra.urdf.xacro-->
-	<!--<xacro:include filename="$(find tegraBot_description)/urdf/turtlebot_common_library.urdf.xacro" />-->
-  <xacro:include filename="$(find tegraBot_description)/urdf/tegraBot_properties.urdf.xacro"/>
-  <xacro:include filename="$(find tegraBot_description)/urdf/kobuki.urdf.xacro" />
-  <xacro:include filename="$(find tegraBot_description)/urdf/stacks/tegraBot_stack.urdf.xacro"/>
-  <xacro:include filename="$(find tegraBot_description)/urdf/computers/m200_jt2.urdf.xacro"/>
-  <xacro:include filename="$(find tegraBot_description)/urdf/sensors/astra.urdf.xacro"/>
-  <xacro:include filename="$(find tegraBot_description)/urdf/sensors/ydlidar_x4.urdf.xacro"/>
+	<!--<xacro:include filename="$(find tegrabot_description)/urdf/turtlebot_common_library.urdf.xacro" />-->
+  <xacro:include filename="$(find tegrabot_description)/urdf/tegraBot_properties.urdf.xacro"/>
+  <xacro:include filename="$(find tegrabot_description)/urdf/kobuki.urdf.xacro" />
+  <xacro:include filename="$(find tegrabot_description)/urdf/stacks/tegraBot_stack.urdf.xacro"/>
+  <xacro:include filename="$(find tegrabot_description)/urdf/computers/m200_jt2.urdf.xacro"/>
+  <xacro:include filename="$(find tegrabot_description)/urdf/sensors/astra.urdf.xacro"/>
+  <xacro:include filename="$(find tegrabot_description)/urdf/sensors/ydlidar_x4.urdf.xacro"/>
   <kobuki/>
   <stack_hexagons parent="base_link"/>
