Commit message: minor model fix

File: urdf/NeuronBot.urdf.xacro (robot description, xacro)
@@ -22,5 +22,5 @@
   <!--<sensor_astra parent="base_link"/>-->
   <sensor_d435 parent="sensor_pole_link">
-	  <origin xyz="0 0 0.6" rpy="0 0 0"/>
+	  <origin xyz="0 0 0.59" rpy="0 0 0"/>
   </sensor_d435>
   <computers parent="plate_middle_link"/>

Commit message: adjust camera angle

File: urdf/NeuronBot.urdf.xacro (robot description, xacro)
@@ -22,5 +22,5 @@
   <!--<sensor_astra parent="base_link"/>-->
   <sensor_d435 parent="sensor_pole_link">
-	  <origin xyz="0 0 0.59" rpy="0 0 0"/>
+	  <origin xyz="0 0 0.59" rpy="0 -0.14 0"/>
   </sensor_d435>
   <computers parent="plate_middle_link"/>
